Commit message: added 4 frames around the hand balls

File: multi_contact_planning/examples/utils/urdf/cogimon.urdf (robot description, URDF)
Before this commit: robot cogimon, 65 links, 64 joints
Links:
- added link l_ball_tip_d
- added link l_ball_tip_l
- added link l_ball_tip_r
- added link l_ball_tip_u
- added link r_ball_tip_d
- added link r_ball_tip_l
- added link r_ball_tip_r
- added link r_ball_tip_u
Joints:
- added joint l_ball_tipj_d: type fixed, parent LBall, child l_ball_tip_d, origin xyz=-0.07 0.0 0.0 rpy=0.0 0.0 0.0
- added joint l_ball_tipj_l: type fixed, parent LBall, child l_ball_tip_l, origin xyz=0.0 0.07 0.0 rpy=0.0 0.0 0.0
- added joint l_ball_tipj_r: type fixed, parent LBall, child l_ball_tip_r, origin xyz=0.0 -0.07 0.0 rpy=0.0 0.0 0.0
- added joint l_ball_tipj_u: type fixed, parent LBall, child l_ball_tip_u, origin xyz=0.07 0.0 0.0 rpy=0.0 0.0 0.0
- added joint r_ball_tipj_d: type fixed, parent RBall, child r_ball_tip_d, origin xyz=-0.07 0.0 0.0 rpy=0.0 0.0 0.0
- added joint r_ball_tipj_l: type fixed, parent RBall, child r_ball_tip_l, origin xyz=0.0 0.07 0.0 rpy=0.0 0.0 0.0
- added joint r_ball_tipj_r: type fixed, parent RBall, child r_ball_tip_r, origin xyz=0.0 -0.07 0.0 rpy=0.0 0.0 0.0
- added joint r_ball_tipj_u: type fixed, parent RBall, child r_ball_tip_u, origin xyz=0.07 0.0 0.0 rpy=0.0 0.0 0.0

Commit message: urdf with frames on hands

File: multi_contact_planning/examples/utils/urdf/cogimon.urdf (robot description, URDF)
Before this commit: robot cogimon, 65 links, 64 joints
Links:
- added link l_ball_tip_d
- added link l_ball_tip_l
- added link l_ball_tip_r
- added link l_ball_tip_u
- added link r_ball_tip_d
- added link r_ball_tip_l
- added link r_ball_tip_r
- added link r_ball_tip_u
Joints:
- added joint l_ball_tipj_d: type fixed, parent LBall, child l_ball_tip_d, origin xyz=-0.07 0.0 -0.01 rpy=0.0 -1.570796326795 0.0
- added joint l_ball_tipj_l: type fixed, parent LBall, child l_ball_tip_l, origin xyz=0.0 0.07 0.0 rpy=0.0 0.0 0.0
- added joint l_ball_tipj_r: type fixed, parent LBall, child l_ball_tip_r, origin xyz=0.0 -0.07 0.0 rpy=0.0 0.0 0.0
- added joint l_ball_tipj_u: type fixed, parent LBall, child l_ball_tip_u, origin xyz=0.07 0.0 0.0 rpy=0.0 0.0 0.0
- added joint r_ball_tipj_d: type fixed, parent RBall, child r_ball_tip_d, origin xyz=-0.07 0.0 -0.01 rpy=0.0 -1.570796326795 0.0
- added joint r_ball_tipj_l: type fixed, parent RBall, child r_ball_tip_l, origin xyz=0.0 0.07 0.0 rpy=0.0 0.0 0.0
- added joint r_ball_tipj_r: type fixed, parent RBall, child r_ball_tip_r, origin xyz=0.0 -0.07 0.0 rpy=0.0 0.0 0.0
- added joint r_ball_tipj_u: type fixed, parent RBall, child r_ball_tip_u, origin xyz=0.07 0.0 0.0 rpy=0.0 0.0 0.0
